Commit message: Oct26_11-43-47_: imitate cassie config

File: legged_gym/resources/robots/biped/urdf/biped.urdf (robot description, URDF)
Before this commit: robot biped, 9 links, 8 joints
Links:
- link abad_R_Link: geometry visual mesh filename=../meshes/abad_right_link.STL
- link hip_R_Link: geometry collision mesh filename=../meshes/hip_right_link.STL; visual mesh filename=../meshes/hip_right_link.STL

Commit message: Oct26_15-44-37_/Oct26_16-51-19_: set self collision
Oct26_15-44-37_：加入self collision，但训不出来

Oct26_16-51-19_：加入self collision，使用Oct26_12-51-17_作为训练checkpoint

File: legged_gym/resources/robots/biped/urdf/biped.urdf (robot description, URDF)
Before this commit: robot biped, 9 links, 8 joints
Links:
- link hip_L_Link: geometry visual mesh filename=../meshes/hip_left_link.STL
- link hip_R_Link: geometry visual mesh filename=../meshes/hip_right_link.STL

Commit message: add depth training and env setup

File: legged_gym/resources/robots/biped/urdf/biped.urdf (robot description, URDF)
Before this commit: robot biped, 9 links, 8 joints
Links:
- added link base; visual box size=0.001 0.001 0.001
- added link camera_box; visual box size=0.025 0.09 0.025
Joints:
- added joint fixed_camera_box: type fixed, parent base, child camera_box, origin xyz=0 0 0 rpy=0 0 0
- added joint floating_base: type fixed, parent base, child base_Link, origin xyz=0 0 0 rpy=0 0 0

Commit message: adaptive play.py to use camera case

File: legged_gym/resources/robots/biped/urdf/biped.urdf (robot description, URDF)
Before this commit: robot biped, 11 links, 10 joints
Links:
- removed link base
Joints:
- removed joint floating_base
- joint fixed_camera_box: parent base -> base_Link

Commit message: optimize model collision with simple geometry

File: legged_gym/resources/robots/biped/urdf/biped.urdf (robot description, URDF)
Before this commit: robot biped, 10 links, 9 joints
Links:
- link abad_L_Link: geometry collision cylinder length=0.05 radius=0.05; visual mesh filename=../meshes/abad_left_link.STL
- link abad_R_Link: geometry collision cylinder length=0.05 radius=0.05; visual mesh filename=../meshes/abad_right_link.STL
- link base_Link: geometry collision box size=0.2 0.3 0.15; visual mesh filename=../meshes/base_link.STL
- link foot_L_Link: geometry collision sphere radius=0.035; visual mesh filename=../meshes/foot_left_link.STL
- link foot_R_Link: geometry collision sphere radius=0.035; visual mesh filename=../meshes/foot_right_link.STL
- link hip_L_Link: geometry collision cylinder length=0.15 radius=0.035; visual mesh filename=../meshes/hip_left_link.STL
- link hip_R_Link: geometry collision cylinder length=0.15 radius=0.035; visual mesh filename=../meshes/hip_right_link.STL
- link knee_L_Link: geometry collision cylinder length=0.26 radius=0.015; visual mesh filename=../meshes/knee_left_link.STL
- link knee_R_Link: geometry collision cylinder length=0.26 radius=0.015; visual mesh filename=../meshes/knee_right_link.STL
